File: kicad_source/OpenCyphalPicoBase.kicad_sch (KiCad schematic)
At the start: 47 parts, among them CN1 RASPBERRYPI_PICO, CN12 S3B-PH-SM4-TB, CN2 SM04B-SRSS-TB, CN3 SM04B-SRSS-TB, CN7 DNI, CN8 DNI, SW1 PTS636 SM43 SMTR LFS, U3 M24C64-RMN6TP

Commit message: corrected BOM
Parts:
- CN8: now left out of the parts list
Changed lines of the file:
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@@
   )
   (symbol (lib_id "Connector_Generic:Conn_02x13_Odd_Even") (at 26.67 71.12 0) (mirror y) (unit 1)
-    (in_bom yes) (on_board yes) (fields_autoplaced)
-    (property "Reference" "CN8" (id 0) (at 25.4 57.15 0))
-    (property "Value" "DNI" (id 1) (at 25.4 59.69 0))
+    (in_bom no) (on_board yes)
+    (property "Reference" "CN8" (id 0) (at 25.4 50.8 0))
+    (property "Value" "DNI" (id 1) (at 25.4 53.34 0))
     (property "Footprint" "Connector_PinHeader_2.54mm:PinHeader_2x13_P2.54mm_Vertical" (id 2) (at 26.67 71.12 0)
       (effects (font (size 1.27 1.27)) hide)
