File: kicad_source/CyphalPicoBase-CAN.kicad_sch (KiCad schematic)
At the start: 47 parts, among them CN1 RASPBERRYPI_PICO, CN12 S3B-PH-SM4-TB, CN2 SM04B-SRSS-TB, CN3 SM04B-SRSS-TB, CN7 DNI, CN8 DNI, SW1 PTS636 SM43 SMTR LFS, U3 M24C64-RMN6TP

Commit message: updated labels in schematic, updated pdf and images
Other:
- title: OpenCyphalPicoBase -> CyphalPicoBase/CAN
Changed lines of the file:
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@@
   (paper "A4")
   (title_block
-    (title "OpenCyphalPicoBase")
-    (date "2023-08-11")
+    (title "CyphalPicoBase/CAN")
+    (date "2023-09-21")
     (rev "0.3")
     (company "generationmake")

Commit message: updated step file of PCB, added JST conectors
Parts:
- CN12: footprint Connector_JST:JST_PH_S3B-PH-SM4-TB_1x03-1MP_P2.00mm_Horizontal -> generationmake:JST_PH_S3B-PH-SM4-TB_1x03-1MP_P2.00mm_Horizontal
- CN2, CN3: footprint Connector_JST:JST_SH_SM04B-SRSS-TB_1x04-1MP_P1.00mm_Horizontal -> generationmake:JST_SH_SM04B-SRSS-TB_1x04-1MP_P1.00mm_Horizontal
Changed lines of the file:
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@@
       (effects (font (size 1.27 1.27)) (justify left))
     )
-    (property "Footprint" "Connector_JST:JST_SH_SM04B-SRSS-TB_1x04-1MP_P1.00mm_Horizontal" (id 2) (at 124.46 135.89 0)
+    (property "Footprint" "generationmake:JST_SH_SM04B-SRSS-TB_1x04-1MP_P1.00mm_Horizontal" (id 2) (at 124.46 135.89 0)
       (effects (font (size 1.27 1.27)) hide)
     )
@@
       (effects (font (size 1.27 1.27)) (justify left))
     )
-    (property "Footprint" "Connector_JST:JST_SH_SM04B-SRSS-TB_1x04-1MP_P1.00mm_Horizontal" (id 2) (at 53.34 170.18 0)
+    (property "Footprint" "generationmake:JST_SH_SM04B-SRSS-TB_1x04-1MP_P1.00mm_Horizontal" (id 2) (at 53.34 170.18 0)
       (effects (font (size 1.27 1.27)) hide)
     )
@@
     (property "Reference" "CN12" (id 0) (at 153.67 87.63 0))
     (property "Value" "S3B-PH-SM4-TB" (id 1) (at 153.67 90.17 0))
-    (property "Footprint" "Connector_JST:JST_PH_S3B-PH-SM4-TB_1x03-1MP_P2.00mm_Horizontal" (id 2) (at 153.67 96.52 0)
+    (property "Footprint" "generationmake:JST_PH_S3B-PH-SM4-TB_1x03-1MP_P2.00mm_Horizontal" (id 2) (at 153.67 96.52 0)
       (effects (font (size 1.27 1.27)) hide)
     )
@@
     )
     (path "/00000000-0000-0000-0000-00006250ded9"
-      (reference "CN2") (unit 1) (value "SM04B-SRSS-TB") (footprint "Connector_JST:JST_SH_SM04B-SRSS-TB_1x04-1MP_P1.00mm_Horizontal")
+      (reference "CN2") (unit 1) (value "SM04B-SRSS-TB") (footprint "generationmake:JST_SH_SM04B-SRSS-TB_1x04-1MP_P1.00mm_Horizontal")
     )
     (path "/00000000-0000-0000-0000-00006250779d"
-      (reference "CN3") (unit 1) (value "SM04B-SRSS-TB") (footprint "Connector_JST:JST_SH_SM04B-SRSS-TB_1x04-1MP_P1.00mm_Horizontal")
+      (reference "CN3") (unit 1) (value "SM04B-SRSS-TB") (footprint "generationmake:JST_SH_SM04B-SRSS-TB_1x04-1MP_P1.00mm_Horizontal")
     )
     (path "/00000000-0000-0000-0000-00005ed92f9c/00000000-0000-0000-0000-000062500ca8"
@@
     )
     (path "/551049a7-4d09-455c-ac39-872acb209e74"
-      (reference "CN12") (unit 1) (value "S3B-PH-SM4-TB") (footprint "Connector_JST:JST_PH_S3B-PH-SM4-TB_1x03-1MP_P2.00mm_Horizontal")
+      (reference "CN12") (unit 1) (value "S3B-PH-SM4-TB") (footprint "generationmake:JST_PH_S3B-PH-SM4-TB_1x03-1MP_P2.00mm_Horizontal")
     )
     (path "/00000000-0000-0000-0000-00005ed92f9c/1c7e72c3-a858-4ad7-b8a5-648cc04b24c6"
